Commit message: added obstacles

File: models/vertical_obst_2.urdf (robot description, URDF)
Before this commit: robot simple_box, 1 links, 0 joints
Links:
- link my_box: geometry collision box size=0.2 0.2 2; visual box size=0.2 0.2 2

File: models/vertical_obst_3.urdf (robot description, URDF)
Before this commit: robot simple_box, 1 links, 0 joints
Links:
- link my_box: geometry collision box size=0.2 0.2 2; visual box size=0.2 0.2 2

File: models/vertical_obst_5.urdf (robot description, URDF)
Before this commit: robot simple_box, 1 links, 0 joints
Links:
- link my_box: geometry collision box size=0.2 0.2 2; visual box size=0.2 0.2 2
